File: hw/sch_pcb/SYMTRANS01.kicad_pcb (KiCad board)
At the start: 2 copper layers, 40.1 x 40.1 mm, 31 parts, among them J1 HEADER_2x04_PARALLEL, J2 HEADER_2x04_PARALLEL, J3 HEADER_1x02, J4 HEADER_1x02, J5 HEADER_1x02, J6 HEADER_1x02, J7 HEADER_2x04_PARALLEL, J8 HEADER_2x04_PARALLEL, M1 HOLE, M2 HOLE, M3 HOLE, M4 HOLE

Commit message: Convert project to KiCAD7.
Other:
- net class Default removed
